File: REZZ-Style_goggles.sch (EAGLE design)
At the start: 79 parts

Commit message: trace adjustments
Parts:
- removed FID1, FID2: FIDUCIAL"", microbuilder:FIDUCIAL""
Changed lines of the file:
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@@
 <part name="C22" library="rcl" deviceset="C-EU" device="C0603"/>
 <part name="JP1" library="NeoPixelRing" deviceset="PINHD-1X1" device="CB"/>
-<part name="FID1" library="microbuilder" deviceset="FIDUCIAL" device="&quot;&quot;"/>
-<part name="FID2" library="microbuilder" deviceset="FIDUCIAL" device="&quot;&quot;"/>
 <part name="JP5" library="NeoPixelRing" deviceset="PINHD-1X1" device="CB"/>
 <part name="JP6" library="NeoPixelRing" deviceset="PINHD-1X1" device="CB"/>
@@
 <instance part="C22" gate="G$1" x="215.9" y="129.54"/>
 <instance part="JP1" gate="G$1" x="17.78" y="76.2" rot="R180"/>
-<instance part="FID1" gate="G$1" x="190.5" y="157.48"/>
-<instance part="FID2" gate="G$1" x="198.12" y="157.48"/>
 <instance part="JP5" gate="G$1" x="30.48" y="104.14" rot="R180"/>
 <instance part="JP6" gate="G$1" x="30.48" y="55.88" rot="R180"/>

Commit message: inner ring completed
Parts:
- added C41, C42, C43, C44: (no value), rcl:C-EUC0603
- added LED41, LED42, LED43, LED44: WS2812B3535, adafruit:WS2812B3535
Connections:
- new net N$42: LED40.DO, LED41.DI
- new net N$43: LED41.DO, LED42.DI
- new net N$44: LED42.DO, LED43.DI
- new net N$45: LED43.DO, LED44.DI
- net GND: now also C41.2, C42.2, C43.2, C44.2, LED41.GND, LED42.GND, LED43.GND, LED44.GND
- net VDD: now also C41.1, C42.1, C43.1, C44.1, LED41.VDD, LED42.VDD, LED43.VDD, LED44.VDD
Changed lines of the file:
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@@
 <part name="C39" library="rcl" deviceset="C-EU" device="C0603"/>
 <part name="C40" library="rcl" deviceset="C-EU" device="C0603"/>
+<part name="LED41" library="adafruit" deviceset="WS2812B" device="3535"/>
+<part name="LED42" library="adafruit" deviceset="WS2812B" device="3535"/>
+<part name="LED43" library="adafruit" deviceset="WS2812B" device="3535"/>
+<part name="LED44" library="adafruit" deviceset="WS2812B" device="3535"/>
+<part name="C41" library="rcl" deviceset="C-EU" device="C0603"/>
+<part name="C42" library="rcl" deviceset="C-EU" device="C0603"/>
+<part name="C43" library="rcl" deviceset="C-EU" device="C0603"/>
+<part name="C44" library="rcl" deviceset="C-EU" device="C0603"/>
 </parts>
 <sheets>
@@
 <instance part="C39" gate="G$1" x="441.96" y="129.54"/>
 <instance part="C40" gate="G$1" x="452.12" y="129.54"/>
+<instance part="LED41" gate="G$1" x="1234.44" y="78.74"/>
+<instance part="LED42" gate="G$1" x="1267.46" y="78.74"/>
+<instance part="LED43" gate="G$1" x="1300.48" y="78.74"/>
+<instance part="LED44" gate="G$1" x="1333.5" y="78.74"/>
+<instance part="C41" gate="G$1" x="462.28" y="129.54"/>
+<instance part="C42" gate="G$1" x="472.44" y="129.54"/>
+<instance part="C43" gate="G$1" x="482.6" y="129.54"/>
+<instance part="C44" gate="G$1" x="492.76" y="129.54"/>
 </instances>
 <busses>
@@
 <junction x="764.54" y="66.04"/>
 <junction x="728.98" y="66.04"/>
+<pinref part="LED41" gate="G$1" pin="GND"/>
+<wire x1="1201.42" y1="66.04" x2="1234.44" y2="66.04" width="0.1524" layer="91"/>
+<wire x1="1234.44" y1="68.58" x2="1234.44" y2="66.04" width="0.1524" layer="91"/>
+<pinref part="LED42" gate="G$1" pin="GND"/>
+<wire x1="1234.44" y1="66.04" x2="1267.46" y2="66.04" width="0.1524" layer="91"/>
+<wire x1="1267.46" y1="68.58" x2="1267.46" y2="66.04" width="0.1524" layer="91"/>
+<pinref part="LED43" gate="G$1" pin="GND"/>
+<wire x1="1267.46" y1="66.04" x2="1300.48" y2="66.04" width="0.1524" layer="91"/>
+<wire x1="1300.48" y1="68.58" x2="1300.48" y2="66.04" width="0.1524" layer="91"/>
+<pinref part="LED44" gate="G$1" pin="GND"/>
+<wire x1="1300.48" y1="66.04" x2="1333.5" y2="66.04" width="0.1524" layer="91"/>
+<wire x1="1333.5" y1="66.04" x2="1333.5" y2="68.58" width="0.1524" layer="91"/>
+<junction x="1234.44" y="66.04"/>
+<junction x="1267.46" y="66.04"/>
+<junction x="1300.48" y="66.04"/>
+<junction x="1333.5" y="66.04"/>
 </segment>
 <segment>
@@
 <junction x="309.88" y="121.92"/>
 <junction x="299.72" y="121.92"/>
+<pinref part="C41" gate="G$1" pin="2"/>
+<wire x1="452.12" y1="121.92" x2="462.28" y2="121.92" width="0.1524" layer="91"/>
+<wire x1="462.28" y1="124.46" x2="462.28" y2="121.92" width="0.1524" layer="91"/>
+<pinref part="C42" gate="G$1" pin="2"/>
+<wire x1="462.28" y1="121.92" x2="472.44" y2="121.92" width="0.1524" layer="91"/>
+<wire x1="472.44" y1="124.46" x2="472.44" y2="121.92" width="0.1524" layer="91"/>
+<pinref part="C43" gate="G$1" pin="2"/>
+<wire x1="472.44" y1="121.92" x2="482.6" y2="121.92" width="0.1524" layer="91"/>
+<wire x1="482.6" y1="124.46" x2="482.6" y2="121.92" width="0.1524" layer="91"/>
+<pinref part="C44" gate="G$1" pin="2"/>
+<wire x1="482.6" y1="121.92" x2="492.76" y2="121.92" width="0.1524" layer="91"/>
+<wire x1="492.76" y1="121.92" x2="492.76" y2="124.46" width="0.1524" layer="91"/>
+<junction x="452.12" y="121.92"/>
+<junction x="462.28" y="121.92"/>
+<junction x="472.44" y="121.92"/>
+<junction x="482.6" y="121.92"/>
+<junction x="492.76" y="121.92"/>
 </segment>
 </net>
@@
 <junction x="1176.02" y="96.52"/>
 <junction x="1206.5" y="96.52"/>
+<pinref part="LED41" gate="G$1" pin="VDD"/>
+<wire x1="1206.5" y1="96.52" x2="1239.52" y2="96.52" width="0.1524" layer="91"/>
+<wire x1="1239.52" y1="93.98" x2="1239.52" y2="96.52" width="0.1524" layer="91"/>
+<pinref part="LED42" gate="G$1" pin="VDD"/>
+<wire x1="1239.52" y1="96.52" x2="1272.54" y2="96.52" width="0.1524" layer="91"/>
+<wire x1="1272.54" y1="93.98" x2="1272.54" y2="96.52" width="0.1524" layer="91"/>
+<pinref part="LED43" gate="G$1" pin="VDD"/>
+<wire x1="1272.54" y1="96.52" x2="1305.56" y2="96.52" width="0.1524" layer="91"/>
+<wire x1="1305.56" y1="93.98" x2="1305.56" y2="96.52" width="0.1524" layer="91"/>
+<pinref part="LED44" gate="G$1" pin="VDD"/>
+<wire x1="1305.56" y1="96.52" x2="1338.58" y2="96.52" width="0.1524" layer="91"/>
+<wire x1="1338.58" y1="96.52" x2="1338.58" y2="93.98" width="0.1524" layer="91"/>
+<junction x="1338.58" y="96.52"/>
+<junction x="1305.56" y="96.52"/>
+<junction x="1272.54" y="96.52"/>
+<junction x="1239.52" y="96.52"/>
 </segment>
 <segment>
@@
 <junction x="431.8" y="134.62"/>
 <junction x="441.96" y="134.62"/>
+<pinref part="C41" gate="G$1" pin="1"/>
+<wire x1="452.12" y1="134.62" x2="462.28" y2="134.62" width="0.1524" layer="91"/>
+<wire x1="462.28" y1="132.08" x2="462.28" y2="134.62" width="0.1524" layer="91"/>
+<pinref part="C42" gate="G$1" pin="1"/>
+<wire x1="462.28" y1="134.62" x2="472.44" y2="134.62" width="0.1524" layer="91"/>
+<wire x1="472.44" y1="132.08" x2="472.44" y2="134.62" width="0.1524" layer="91"/>
+<pinref part="C43" gate="G$1" pin="1"/>
+<wire x1="472.44" y1="134.62" x2="482.6" y2="134.62" width="0.1524" layer="91"/>
+<wire x1="482.6" y1="132.08" x2="482.6" y2="134.62" width="0.1524" layer="91"/>
+<pinref part="C44" gate="G$1" pin="1"/>
+<wire x1="482.6" y1="134.62" x2="492.76" y2="134.62" width="0.1524" layer="91"/>
+<wire x1="492.76" y1="134.62" x2="492.76" y2="132.08" width="0.1524" layer="91"/>
+<junction x="452.12" y="134.62"/>
+<junction x="462.28" y="134.62"/>
+<junction x="472.44" y="134.62"/>
+<junction x="482.6" y="134.62"/>
+<junction x="492.76" y="134.62"/>
 </segment>
 </net>
@@
 </segment>
 </net>
+<net name="N$42" class="0">
+<segment>
+<pinref part="LED40" gate="G$1" pin="DO"/>
+<pinref part="LED41" gate="G$1" pin="DI"/>
+<wire x1="1214.12" y1="76.2" x2="1221.74" y2="76.2" width="0.1524" layer="91"/>
+</segment>
+</net>
+<net name="N$43" class="0">
+<segment>
+<pinref part="LED41" gate="G$1" pin="DO"/>
+<pinref part="LED42" gate="G$1" pin="DI"/>
+<wire x1="1247.14" y1="76.2" x2="1254.76" y2="76.2" width="0.1524" layer="91"/>
+</segment>
+</net>
+<net name="N$44" class="0">
+<segment>
+<pinref part="LED42" gate="G$1" pin="DO"/>
+<pinref part="LED43" gate="G$1" pin="DI"/>
+<wire x1="1280.16" y1="76.2" x2="1287.78" y2="76.2" width="0.1524" layer="91"/>
+</segment>
+</net>
+<net name="N$45" class="0">
+<segment>
+<pinref part="LED43" gate="G$1" pin="DO"/>
+<pinref part="LED44" gate="G$1" pin="DI"/>
+<wire x1="1313.18" y1="76.2" x2="1320.8" y2="76.2" width="0.1524" layer="91"/>
+</segment>
+</net>

Commit message: revised pads, adjusted silk screen
Parts:
- removed JP1, JP3, JP4, JP5, JP6: (no value), NeoPixelRing:PINHD-1X1CB
- added GND, INPUT, VDD: WIREPADSMD1,27-254, wirepad:WIREPADSMD1,27-254
Connections:
- net GND: now also GND.P; no longer JP4.1, JP6.1
- net N$26: now also INPUT.P; no longer JP1.1
- net VDD: now also VDD.P; no longer JP3.1, JP5.1
Changed lines of the file:
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@@
 <?xml version="1.0" encoding="utf-8"?>
 <!DOCTYPE eagle SYSTEM "eagle.dtd">
-<eagle version="7.3.0">
+<eagle version="7.7.0">
 <drawing>
 <settings>
@@
 <part name="VDD1" library="supply1" deviceset="VDD" device=""/>
 <part name="VDD2" library="supply1" deviceset="VDD" device=""/>
-<part name="JP3" library="NeoPixelRing" deviceset="PINHD-1X1" device="CB"/>
-<part name="JP4" library="NeoPixelRing" deviceset="PINHD-1X1" device="CB"/>
 <part name="LED13" library="adafruit" deviceset="WS2812B" device="3535"/>
 <part name="LED14" library="adafruit" deviceset="WS2812B" device="3535"/>
@@
 <part name="C21" library="rcl" deviceset="C-EU" device="C0603"/>
 <part name="C22" library="rcl" deviceset="C-EU" device="C0603"/>
-<part name="JP1" library="NeoPixelRing" deviceset="PINHD-1X1" device="CB"/>
-<part name="JP5" library="NeoPixelRing" deviceset="PINHD-1X1" device="CB"/>
-<part name="JP6" library="NeoPixelRing" deviceset="PINHD-1X1" device="CB"/>
 <part name="R1" library="microbuilder" deviceset="RESISTOR" device="_0603_NOOUT"/>
 <part name="LED25" library="adafruit" deviceset="WS2812B" device="3535"/>
@@
 <part name="C43" library="rcl" deviceset="C-EU" device="C0603"/>
 <part name="C44" library="rcl" deviceset="C-EU" device="C0603"/>
+<part name="VDD" library="wirepad" deviceset="WIREPAD" device="SMD1,27-254"/>
+<part name="INPUT" library="wirepad" deviceset="WIREPAD" device="SMD1,27-254"/>
+<part name="GND" library="wirepad" deviceset="WIREPAD" device="SMD1,27-254"/>
 </parts>
 <sheets>
@@
 <instance part="VDD1" gate="G$1" x="365.76" y="101.6"/>
 <instance part="VDD2" gate="G$1" x="165.1" y="139.7"/>
-<instance part="JP3" gate="G$1" x="30.48" y="96.52" rot="R180"/>
-<instance part="JP4" gate="G$1" x="30.48" y="66.04" rot="R180"/>
 <instance part="LED13" gate="G$1" x="388.62" y="78.74"/>
 <instance part="LED14" gate="G$1" x="416.56" y="78.74"/>
@@
 <instance part="C21" gate="G$1" x="175.26" y="129.54"/>
 <instance part="C22" gate="G$1" x="215.9" y="129.54"/>
-<instance part="JP1" gate="G$1" x="17.78" y="76.2" rot="R180"/>
-<instance part="JP5" gate="G$1" x="30.48" y="104.14" rot="R180"/>
-<instance part="JP6" gate="G$1" x="30.48" y="55.88" rot="R180"/>
 <instance part="R1" gate="G$1" x="33.02" y="76.2"/>
 <instance part="LED25" gate="G$1" x="728.98" y="78.74"/>
@@
 <instance part="C43" gate="G$1" x="482.6" y="129.54"/>
 <instance part="C44" gate="G$1" x="492.76" y="129.54"/>
+<instance part="VDD" gate="G$1" x="15.24" y="96.52"/>
+<instance part="INPUT" gate="G$1" x="10.16" y="76.2"/>
+<instance part="GND" gate="G$1" x="25.4" y="55.88"/>
 </instances>
 <busses>
@@
 <wire x1="81.28" y1="66.04" x2="53.34" y2="66.04" width="0.1524" layer="91"/>
 <wire x1="53.34" y1="66.04" x2="53.34" y2="68.58" width="0.1524" layer="91"/>
-<pinref part="JP4" gate="G$1" pin="1"/>
-<wire x1="33.02" y1="66.04" x2="53.34" y2="66.04" width="0.1524" layer="91"/>
 <pinref part="LED24" gate="G$1" pin="GND"/>
 <wire x1="360.68" y1="66.04" x2="388.62" y2="66.04" width="0.1524" layer="91"/>
@@
 <junction x="668.02" y="66.04"/>
 <junction x="695.96" y="66.04"/>
-<pinref part="JP6" gate="G$1" pin="1"/>
-<wire x1="33.02" y1="55.88" x2="53.34" y2="55.88" width="0.1524" layer="91"/>
+<wire x1="27.94" y1="55.88" x2="53.34" y2="55.88" width="0.1524" layer="91"/>
 <wire x1="53.34" y1="55.88" x2="53.34" y2="66.04" width="0.1524" layer="91"/>
 <wire x1="695.96" y1="66.04" x2="728.98" y2="66.04" width="0.1524" layer="91"/>
@@
 <junction x="1300.48" y="66.04"/>
 <junction x="1333.5" y="66.04"/>
+<pinref part="GND" gate="G$1" pin="P"/>
 </segment>
 <segment>
@@
 <wire x1="114.3" y1="96.52" x2="86.36" y2="96.52" width="0.1524" layer="91"/>
 <wire x1="86.36" y1="96.52" x2="58.42" y2="96.52" width="0.1524" layer="91"/>
-<wire x1="58.42" y1="96.52" x2="50.8" y2="96.52" width="0.1524" layer="91"/>
 <pinref part="LED1" gate="G$1" pin="VDD"/>
 <wire x1="58.42" y1="93.98" x2="58.42" y2="96.52" width="0.1524" layer="91"/>
@@
 <pinref part="LED11" gate="G$1" pin="VDD"/>
 <wire x1="337.82" y1="93.98" x2="337.82" y2="96.52" width="0.1524" layer="91"/>
-<pinref part="JP3" gate="G$1" pin="1"/>
-<wire x1="33.02" y1="96.52" x2="50.8" y2="96.52" width="0.1524" layer="91"/>
+<wire x1="17.78" y1="96.52" x2="58.42" y2="96.52" width="0.1524" layer="91"/>
 <pinref part="LED24" gate="G$1" pin="VDD"/>
 <wire x1="365.76" y1="96.52" x2="393.7" y2="96.52" width="0.1524" layer="91"/>
@@
 <wire x1="393.7" y1="93.98" x2="393.7" y2="96.52" width="0.1524" layer="91"/>
 <junction x="365.76" y="96.52"/>
-<junction x="50.8" y="96.52"/>
 <junction x="58.42" y="96.52"/>
 <junction x="86.36" y="96.52"/>
@@
 <junction x="673.1" y="96.52"/>
 <junction x="701.04" y="96.52"/>
-<pinref part="JP5" gate="G$1" pin="1"/>
-<wire x1="33.02" y1="104.14" x2="50.8" y2="104.14" width="0.1524" layer="91"/>
-<wire x1="50.8" y1="104.14" x2="50.8" y2="96.52" width="0.1524" layer="91"/>
 <wire x1="701.04" y1="96.52" x2="734.06" y2="96.52" width="0.1524" layer="91"/>
 <pinref part="LED25" gate="G$1" pin="VDD"/>
@@
 <junction x="1272.54" y="96.52"/>
 <junction x="1239.52" y="96.52"/>
+<pinref part="VDD" gate="G$1" pin="P"/>
 </segment>
 <segment>
@@
 <net name="N$26" class="0">
 <segment>
-<pinref part="JP1" gate="G$1" pin="1"/>
-<wire x1="20.32" y1="76.2" x2="27.94" y2="76.2" width="0.1524" layer="91"/>
+<wire x1="12.7" y1="76.2" x2="27.94" y2="76.2" width="0.1524" layer="91"/>
 <pinref part="R1" gate="G$1" pin="1"/>
-</segment>
-</net>
+<pinref part="INPUT" gate="G$1" pin="P"/>
+</segment>
+</net>
